File: Board.sch (EAGLE design)
At the start: 0 parts

Commit message: add m5 atom martix component
Parts:
- added M5-ATOM1: (no value), Design-by-Amri:M5-ATOM-MATRIX
Changed lines of the file:
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@@
 <layer number="51" name="tDocu" color="7" fill="1" visible="no" active="no"/>
 <layer number="52" name="bDocu" color="7" fill="1" visible="no" active="no"/>
+<layer number="88" name="SimResults" color="9" fill="1" visible="yes" active="yes"/>
+<layer number="89" name="SimProbes" color="9" fill="1" visible="yes" active="yes"/>
 <layer number="90" name="Modules" color="5" fill="1" visible="yes" active="yes"/>
 <layer number="91" name="Nets" color="2" fill="1" visible="yes" active="yes"/>
@@
 </classes>
 <parts>
-<part name="FRAME1" library="frames" deviceset="A5L-LOC" device=""/>
+<part name="FRAME1" library="frames" library_urn="urn:adsk.eagle:library:229" deviceset="A5L-LOC" device=""/>
+<part name="M5-ATOM1" library="Design-by-Amri" deviceset="M5-ATOM" device="-MATRIX"/>
 </parts>
 <sheets>
@@
 <instance part="FRAME1" gate="G$1" x="22.86" y="-7.62" smashed="yes">
 <attribute name="SHEET" x="177.165" y="-2.54" size="2.54" layer="94"/>
+</instance>
+<instance part="M5-ATOM1" gate="G$1" x="101.6" y="81.28" smashed="yes">
+<attribute name="NAME" x="91.948" y="89.408" size="1.27" layer="95"/>
 </instance>
 </instances>
@@
 </schematic>
 </drawing>
+<compatibility>
+<note version="8.2" severity="warning">
+Since Version 8.2, EAGLE supports online libraries. The ids
+of those online libraries will not be understood (or retained)
+with this version.
+</note>
+<note version="8.3" severity="warning">
+Since Version 8.3, EAGLE supports URNs for individual library
+assets (packages, symbols, and devices). The URNs of those assets
+will not be understood (or retained) with this version.
+</note>
+</compatibility>
 </eagle>
